File: circuit/circuit.kicad_sch (KiCad schematic)
At the start: 0 parts

Commit message: .
Parts:
- added U1: Pico, RPi_Pico:RPi_Pico_SMD_TH, symbol MCU_RaspberryPi_and_Boards:Pico
Changed lines of the file:
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@@
 (kicad_sch (version 20230121) (generator eeschema)
   (paper "A4")
+  (symbol (lib_id "MCU_RaspberryPi_and_Boards:Pico") (at 134.62 82.55 0) (unit 1)
+    (in_bom yes) (on_board yes) (dnp no) (fields_autoplaced)
+    (property "Reference" "U1" (at 134.62 50.8 0)
+      (effects (font (size 1.27 1.27)))
+    )
+    (property "Value" "Pico" (at 134.62 53.34 0)
+      (effects (font (size 1.27 1.27)))
+    )
+    (property "Footprint" "RPi_Pico:RPi_Pico_SMD_TH" (at 134.62 82.55 90)
+      (effects (font (size 1.27 1.27)) hide)
+    )
+    (property "Datasheet" "" (at 134.62 82.55 0)
+      (effects (font (size 1.27 1.27)) hide)
+    )
+    (pin "1")
+    (pin "10")
+    (pin "11")
+    (pin "12")
+    (pin "13")
+    (pin "14")
+    (pin "15")
+    (pin "16")
+    (pin "17")
+    (pin "18")
+    (pin "19")
+    (pin "2")
+    (pin "20")
+    (pin "21")
+    (pin "22")
+    (pin "23")
+    (pin "24")
+    (pin "25")
+    (pin "26")
+    (pin "27")
+    (pin "28")
+    (pin "29")
+    (pin "3")
+    (pin "30")
+    (pin "31")
+    (pin "32")
+    (pin "33")
+    (pin "34")
+    (pin "35")
+    (pin "36")
+    (pin "37")
+    (pin "38")
+    (pin "39")
+    (pin "4")
+    (pin "40")
+    (pin "41")
+    (pin "42")
+    (pin "43")
+    (pin "5")
+    (pin "6")
+    (pin "7")
+    (pin "8")
+    (pin "9")
+    (instances
+      (project "circuit"
+        (path "/0a6b6e71-7152-4192-b04d-e2f91e81ba3a"
+          (reference "U1") (unit 1)
+        )
+      )
+    )
+  )
   (sheet_instances
     (path "/" (page "1"))
